File: raven-main/power.kicad_sch (KiCad schematic)
At the start: 43 parts, among them Q1 SQJQ100EL, T1 Transformer_1P_1S, U3 LM66200DRLR, U4 MAX77827AEFD+T, U5 SC4215ASTRT, U6 LM5185QPWPRQ1, U7 TPS7A4701xRGW

Commit message: Added missing resistor values
Parts:
- R23: value R -> 10.7k
- R24: value R -> 100
- R25: value R -> 20m
Changed lines of the file:
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@@
 			)
 		)
-		(property "Value" "R"
+		(property "Value" "10.7k"
 			(at 118.11 134.62 90)
 			(show_name no)
@@
 			)
 		)
-		(property "Value" "R"
+		(property "Value" "20m"
 			(at 138.43 166.3699 0)
 			(show_name no)
@@
 			)
 		)
-		(property "Value" "R"
+		(property "Value" "100"
 			(at 128.27 151.13 90)
 			(show_name no)
