File: raven-main/Detector-Breakout-Board/detector.kicad_sch (KiCad schematic)
At the start: 27 parts, among them IC1 ADA4817-1ARDZ-R7, IC2 ADA4817-1ARDZ-R7, U10 TLV3201AIDCKT, U9 TLV3201AIDCKT

Commit message: Changed detector output to 3.3V
Connections:
- net +5V: no longer C37.2, C44.2, U10.5 (VCC), U9.5 (VCC)
- new net +3V3: C37.2, C44.2, U10.5 (VCC), U9.5 (VCC)
Changed lines of the file:
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@@
 			)
 		)
-		(property "Value" "+5V"
+		(property "Value" "+3V3"
 			(at 226.06 133.35 0)
 			(show_name no)
@@
 			)
 		)
-		(property "Value" "+5V"
-			(at 223.52 54.61 0)
-			(show_name no)
-			(do_not_autoplace no)
-			(effects
-				(font
-					(size 1.27 1.27)
-				)
-			)
-		)
+		(property "Value" "+3V3"
+			(at 226.06 58.4199 0)
+			(show_name no)
+			(do_not_autoplace no)
+			(effects
+				(font
+					(size 1.27 1.27)
+				)
+				(justify left)
+			)
+		)
