File: raven-main/Detector-Breakout-Board/_restore_backup_2026-07-21T18-53-36-536/power.kicad_sch (KiCad schematic)
At the start: 31 parts, among them J1 DeployLipo, J9 UCLipo, Q1 SQJQ100EL, T1 Transformer_1P_1S, U6 LM5185QPWPRQ1, U7 TPS7A4701xRGW, U8 TPS7A4701xRGW

Commit message: Updated pcb layout
Parts:
- T1: footprint Transistor_Power:GaN_Systems_GaNPX-3_5x6.6mm_Drain2.93x0.6mm -> Transformer_THT:Transformer_37x44
- U6: footprint footprints:PWP0014G-IPC_A -> PWP0014G-IPC_A
Changed lines of the file:
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@@
 			)
 		)
-		(property "Footprint" "Transistor_Power:GaN_Systems_GaNPX-3_5x6.6mm_Drain2.93x0.6mm"
+		(property "Footprint" "Transformer_THT:Transformer_37x44"
 			(at 144.78 93.98 0)
 			(hide yes)
@@
 			)
 		)
-		(property "Footprint" "footprints:PWP0014G-IPC_A"
+		(property "Footprint" "PWP0014G-IPC_A"
 			(at 71.12 109.22 0)
 			(hide yes)
