File: raven-main/Detector-Power-Board/_restore_backup_2026-07-30T17-38-07-352/detector-power.kicad_pcb (KiCad board)
At the start: 2 copper layers, 37 x 52.5 mm, 36 parts, among them J1 DeployLipo, J2 Conn_01x06, J9 UCLipo, U1 STPS20M100SG-TR, U6 LM5185QPWPRQ1, U7 TPS7A4701xRGW, U8 TPS7A4701xRGW

Commit message: Added transformer, diode and mosfet
Parts:
- moved U8 12.8 mm to (129.8, 95.8)
- moved C46 12.4 mm to (135.5, 97.5), turned to 0 degrees
- moved 1 12.0 mm to (122.5, 93.3)
- moved U1 11.6 mm to (128.2, 107.9), turned to 90 degrees
- moved R39 10.7 mm to (135.5, 95.8), turned to 0 degrees
- moved H104 8.91 mm to (116.0, 97.0)
- moved H103 8.84 mm to (142.5, 97.0)
- moved R38 8.46 mm to (135.5, 93.0), turned to 180 degrees
- moved TR1 2.81 mm to (118.0, 83.1)
- moved J2 2.56 mm to (143.0, 71.5)
Routing:
- net GND: track 201.2 -> 175.8 mm, vias 16 -> 14
- net Net-(1-Gate): track 44.1 -> 27.7 mm
- net /Power_Out_50V: track 55.0 -> 41.0 mm, vias 4 -> 2
- net Net-(R26-Pad1): track 27.4 -> 17.1 mm
- net Net-(U8-SENSE/FB): track 12.1 -> 21.0 mm, vias 0 -> 4
- net Net-(1-Drain): track 40.8 -> 32.6 mm, vias 4 -> 2
- net Net-(1-Source): track 34.1 -> 27.2 mm
- net /Data_In_5V: track 32.2 -> 26.8 mm, vias 4 -> 3
- net /BBIN: track 77.8 -> 82.6 mm, vias 8 -> 7
- net /ON-OFF: track 54.5 -> 51.8 mm, vias 4 -> 3
- net /Data_Out_3V3: track 29.2 -> 27.5 mm
- net Net-(U8-NR): track 5.51 -> 4.41 mm, vias 0 -> 2
- net /Power_Out_5V: track 29.8 -> 28.9 mm
Other:
- board size 37 x 52.5 mm -> 37 x 44.5 mm
