File: raven-main/Detector-Power-Board/detector-power.kicad_pcb (KiCad board)
At the start: 2 copper layers, 37 x 52.5 mm, 45 parts, among them J1 DeployLipo, J2 Conn_01x06, J9 UCLipo, Q1 CSD18543Q3A, Q2 CSD18543Q3A, U2 TPS43060RTE, U7 TPS7A4701xRGW, U8 TPS7A4701xRGW

Commit message: Added corrected deco detials
Other:
- board text added: "Payload 2026"
- board text added: "Power Board for HARRIER v1.0"
- board text added: "Power board for Harrier v1.0 2026"
- board text removed: "Power Board for HARRIER v.1 2026"
- board text removed: "Power board for Harrier v.1 2026"
Changed lines of the file:
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@@
 		(layer "Edge.Cuts")
 	)
-	(gr_text "Power board for Harrier v.1 2026"
+	(gr_text "Power board for Harrier v1.0 2026"
 		(at 119 108 0)
 		(layer "F.SilkS")
@@
 			)
 			(justify left bottom)
+		)
+	)
+	(gr_text "Payload 2026"
+		(at 135 100 0)
+		(layer "B.SilkS")
+		(effects
+			(font
+				(size 1 1)
+				(thickness 0.1)
+			)
+			(justify left bottom mirror)
 		)
 	)
@@
 		)
 	)
-	(gr_text "Power Board for HARRIER v.1 2026"
-		(at 142 96 0)
+	(gr_text "Power Board for HARRIER v1.0"
+		(at 141 96 0)
 		(layer "B.SilkS")
 		(effects
